Commit message: Improve paint diagnostics, collision recovery, workcell profiles and platform appearance
git-svn-id: https://192.168.2.101:8443/svn/25488_ZeroErr/trunk@89 4fd3d927-d0b4-2643-a258-f5eadda0d283

File: backend/ros2_ws/eRob_moveit/src/eRob_ROS2_MoveIt/zeroerr/config/paint/urdfs/erob_arm_small.urdf (robot description, URDF)
Before this commit: robot eRobo3, 13 links, 12 joints
Links:
- link Link_1: geometry collision mesh filename=package://zeroerr/meshes/robots/zeroerr/common/Link_1.stl scale=1.00000 1.00000 1.00000; visual mesh filename=package://zeroerr/meshes/robots/zeroerr/common/Link_1.stl scale=1.00000 1.00000 1.00000
- link Link_2: geometry collision mesh filename=package://zeroerr/meshes/robots/zeroerr/extended_links/Link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 scale=1.00000 1.00000 1.00000; visual mesh filename=package://zeroerr/meshes/robots/zeroerr/extended_links/Link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 scale=1.00000 1.00000 1.00000
- link Link_3: geometry collision mesh filename=package://zeroerr/meshes/robots/zeroerr/extended_links/Link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 scale=1.00000 1.00000 1.00000; visual mesh filename=package://zeroerr/meshes/robots/zeroerr/extended_links/Link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 scale=1.00000 1.00000 1.00000
- link Link_4: geometry collision mesh filename=package://zeroerr/meshes/robots/zeroerr/common/Link_4.stl scale=1.00000 1.00000 1.00000; visual mesh filename=package://zeroerr/meshes/robots/zeroerr/common/Link_4.stl scale=1.00000 1.00000 1.00000
- link Link_5: geometry collision mesh filename=package://zeroerr/meshes/robots/zeroerr/common/Link_5.stl scale=1.00000 1.00000 1.00000; visual mesh filename=package://zeroerr/meshes/robots/zeroerr/common/Link_5.stl scale=1.00000 1.00000 1.00000
- link Link_6: geometry collision mesh filename=package://zeroerr/meshes/robots/zeroerr/common/Link_6.stl scale=1.00000 1.00000 1.00000; visual mesh filename=package://zeroerr/meshes/robots/zeroerr/common/Link_6.stl scale=1.00000 1.00000 1.00000
- link base_link_inertial: geometry collision mesh filename=package://zeroerr/meshes/robots/zeroerr/common/base_link.stl scale=1.00000 1.00000 1.00000; visual mesh filename=package://zeroerr/meshes/robots/zeroerr/common/base_link.stl scale=1.00000 1.00000 1.00000
- link tool0: geometry collision mesh filename=package://zeroerr/meshes/tools/pointer/ToolPointer.stl scale=0.001 0.001 0.001; visual mesh filename=package://zeroerr/meshes/tools/pointer/ToolPointer.stl scale=0.001 0.001 0.001

File: backend/ros2_ws/eRob_moveit/src/eRob_ROS2_MoveIt/zeroerr/config/paint/urdfs/erob_arm_small.with_mounting_stl.urdf (robot description, URDF)
Before this commit: robot eRobo3, 12 links, 11 joints
Links:
- link Link_1: geometry collision mesh filename=package://zeroerr/meshes/robots/zeroerr/common/Link_1.stl scale=1.00000 1.00000 1.00000; visual mesh filename=package://zeroerr/meshes/robots/zeroerr/common/Link_1.stl scale=1.00000 1.00000 1.00000
- link Link_2: geometry collision mesh filename=package://zeroerr/meshes/robots/zeroerr/extended_links/Link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 scale=1.00000 1.00000 1.00000; visual mesh filename=package://zeroerr/meshes/robots/zeroerr/extended_links/Link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 scale=1.00000 1.00000 1.00000
- link Link_3: geometry collision mesh filename=package://zeroerr/meshes/robots/zeroerr/extended_links/Link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 scale=1.00000 1.00000 1.00000; visual mesh filename=package://zeroerr/meshes/robots/zeroerr/extended_links/Link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 scale=1.00000 1.00000 1.00000
- link Link_4: geometry collision mesh filename=package://zeroerr/meshes/robots/zeroerr/common/Link_4.stl scale=1.00000 1.00000 1.00000; visual mesh filename=package://zeroerr/meshes/robots/zeroerr/common/Link_4.stl scale=1.00000 1.00000 1.00000
- link Link_5: geometry collision mesh filename=package://zeroerr/meshes/robots/zeroerr/common/Link_5.stl scale=1.00000 1.00000 1.00000; visual mesh filename=package://zeroerr/meshes/robots/zeroerr/common/Link_5.stl scale=1.00000 1.00000 1.00000
- link Link_6: geometry collision mesh filename=package://zeroerr/meshes/robots/zeroerr/common/Link_6.stl scale=1.00000 1.00000 1.00000; visual mesh filename=package://zeroerr/meshes/robots/zeroerr/common/Link_6.stl scale=1.00000 1.00000 1.00000
- link base_link_inertial: geometry collision mesh filename=package://zeroerr/meshes/robots/zeroerr/common/base_link.stl scale=1.00000 1.00000 1.00000; visual mesh filename=package://zeroerr/meshes/robots/zeroerr/common/base_link.stl scale=1.00000 1.00000 1.00000
- link mounting_surface: geometry collision box size=0.007 0.207 0.008; collision box size=0.007 0.532 0.008
- link tool0: geometry collision mesh filename=package://zeroerr/meshes/tools/disk_centered/00035513_disk_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 scale=0.001 0.001 0.001; visual mesh filename=package://zeroerr/meshes/tools/disk_centered/00035513_disk_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 scale=0.001 0.001 0.001

File: backend/ros2_ws/eRob_moveit/src/eRob_ROS2_MoveIt/zeroerr/config/paint_short_links/urdfs/erob_arm_short_links.with_mounting_stl.urdf (robot description, URDF)
Before this commit: robot eRobo3, 12 links, 11 joints
Links:
- link Link_1: geometry collision mesh filename=package://zeroerr/meshes/robots/zeroerr/common/Link_1.stl scale=1.00000 1.00000 1.00000; visual mesh filename=package://zeroerr/meshes/robots/zeroerr/common/Link_1.stl scale=1.00000 1.00000 1.00000
- link Link_2: geometry collision mesh filename=package://zeroerr/meshes/robots/zeroerr/short_links/Link_2.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 scale=1.00000 1.00000 1.00000; visual mesh filename=package://zeroerr/meshes/robots/zeroerr/short_links/Link_2.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 scale=1.00000 1.00000 1.00000
- link Link_3: geometry collision mesh filename=package://zeroerr/meshes/robots/zeroerr/short_links/Link_3.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 scale=1.00000 1.00000 1.00000; visual mesh filename=package://zeroerr/meshes/robots/zeroerr/short_links/Link_3.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 scale=1.00000 1.00000 1.00000
- link Link_4: geometry collision mesh filename=package://zeroerr/meshes/robots/zeroerr/common/Link_4.stl scale=1.00000 1.00000 1.00000; visual mesh filename=package://zeroerr/meshes/robots/zeroerr/common/Link_4.stl scale=1.00000 1.00000 1.00000
- link Link_5: geometry collision mesh filename=package://zeroerr/meshes/robots/zeroerr/common/Link_5.stl scale=1.00000 1.00000 1.00000; visual mesh filename=package://zeroerr/meshes/robots/zeroerr/common/Link_5.stl scale=1.00000 1.00000 1.00000
- link Link_6: geometry collision mesh filename=package://zeroerr/meshes/robots/zeroerr/common/Link_6.stl scale=1.00000 1.00000 1.00000; visual mesh filename=package://zeroerr/meshes/robots/zeroerr/common/Link_6.stl scale=1.00000 1.00000 1.00000
- link base_link_inertial: geometry collision mesh filename=package://zeroerr/meshes/robots/zeroerr/common/base_link.stl scale=1.00000 1.00000 1.00000; visual mesh filename=package://zeroerr/meshes/robots/zeroerr/common/base_link.stl scale=1.00000 1.00000 1.00000
- link tool0: geometry collision mesh filename=package://zeroerr/meshes/tools/pointer/ToolPointer.stl scale=0.001 0.001 0.001; visual mesh filename=package://zeroerr/meshes/tools/pointer/ToolPointer.stl scale=0.001 0.001 0.001

File: backend/ros2_ws/eRob_moveit/src/eRob_ROS2_MoveIt/zeroerr/config/urdfs/erob_arm.urdf (robot description, URDF)
Before this commit: robot eRobo3, 12 links, 11 joints
Links:
- link Link_1: geometry collision mesh filename=package://zeroerr/meshes/robots/zeroerr/common/Link_1.stl scale=1.00000 1.00000 1.00000; visual mesh filename=package://zeroerr/meshes/robots/zeroerr/common/Link_1.stl scale=1.00000 1.00000 1.00000
- link Link_2: geometry collision mesh filename=package://zeroerr/meshes/robots/zeroerr/short_links/Link_2.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 scale=1.00000 1.00000 1.00000; visual mesh filename=package://zeroerr/meshes/robots/zeroerr/short_links/Link_2.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 scale=1.00000 1.00000 1.00000
- link Link_3: geometry collision mesh filename=package://zeroerr/meshes/robots/zeroerr/short_links/Link_3.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 scale=1.00000 1.00000 1.00000; visual mesh filename=package://zeroerr/meshes/robots/zeroerr/short_links/Link_3.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 scale=1.00000 1.00000 1.00000
- link Link_4: geometry collision mesh filename=package://zeroerr/meshes/robots/zeroerr/common/Link_4.stl scale=1.00000 1.00000 1.00000; visual mesh filename=package://zeroerr/meshes/robots/zeroerr/common/Link_4.stl scale=1.00000 1.00000 1.00000
- link Link_5: geometry collision mesh filename=package://zeroerr/meshes/robots/zeroerr/common/Link_5.stl scale=1.00000 1.00000 1.00000; visual mesh filename=package://zeroerr/meshes/robots/zeroerr/common/Link_5.stl scale=1.00000 1.00000 1.00000
- link Link_6: geometry collision mesh filename=package://zeroerr/meshes/robots/zeroerr/common/Link_6.stl scale=1.00000 1.00000 1.00000; visual mesh filename=package://zeroerr/meshes/robots/zeroerr/common/Link_6.stl scale=1.00000 1.00000 1.00000
- link base_link_inertial: geometry collision mesh filename=package://zeroerr/meshes/robots/zeroerr/common/base_link.stl scale=1.00000 1.00000 1.00000; visual mesh filename=package://zeroerr/meshes/robots/zeroerr/common/base_link.stl scale=1.00000 1.00000 1.00000
- link disk_link: geometry collision mesh filename=package://zeroerr/meshes/tools/welding_disk/disk.stl scale=0.001 0.001 0.001; visual mesh filename=package://zeroerr/meshes/tools/welding_disk/disk.stl scale=0.001 0.001 0.001

File: backend/ros2_ws/eRob_moveit/src/eRob_ROS2_MoveIt/zeroerr/config/urdfs/erob_arm_backup_corrected_mass.urdf (robot description, URDF)
Before this commit: robot eRobo3, 12 links, 11 joints
Links:
- link Link_1: geometry collision mesh filename=package://zeroerr/meshes/robots/zeroerr/common/Link_1.stl scale=1.00000 1.00000 1.00000; visual mesh filename=package://zeroerr/meshes/robots/zeroerr/common/Link_1.stl scale=1.00000 1.00000 1.00000
- link Link_2: geometry collision mesh filename=package://zeroerr/meshes/robots/zeroerr/extended_links/Link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 scale=1.00000 1.00000 1.00000; visual mesh filename=package://zeroerr/meshes/robots/zeroerr/extended_links/Link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 scale=1.00000 1.00000 1.00000
- link Link_3: geometry collision mesh filename=package://zeroerr/meshes/robots/zeroerr/extended_links/Link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 scale=1.00000 1.00000 1.00000; visual mesh filename=package://zeroerr/meshes/robots/zeroerr/extended_links/Link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 scale=1.00000 1.00000 1.00000
- link Link_4: geometry collision mesh filename=package://zeroerr/meshes/robots/zeroerr/common/Link_4.stl scale=1.00000 1.00000 1.00000; visual mesh filename=package://zeroerr/meshes/robots/zeroerr/common/Link_4.stl scale=1.00000 1.00000 1.00000
- link Link_5: geometry collision mesh filename=package://zeroerr/meshes/robots/zeroerr/common/Link_5.stl scale=1.00000 1.00000 1.00000; visual mesh filename=package://zeroerr/meshes/robots/zeroerr/common/Link_5.stl scale=1.00000 1.00000 1.00000
- link Link_6: geometry collision mesh filename=package://zeroerr/meshes/robots/zeroerr/common/Link_6.stl scale=1.00000 1.00000 1.00000; visual mesh filename=package://zeroerr/meshes/robots/zeroerr/common/Link_6.stl scale=1.00000 1.00000 1.00000
- link base_link_inertial: geometry collision mesh filename=package://zeroerr/meshes/robots/zeroerr/common/base_link.stl scale=1.00000 1.00000 1.00000; visual mesh filename=package://zeroerr/meshes/robots/zeroerr/common/base_link.stl scale=1.00000 1.00000 1.00000
- link ring_raster_m5: geometry collision mesh filename=package://zeroerr/meshes/tools/welding_disk/disk.stl scale=0.001 0.001 0.001; visual mesh filename=package://zeroerr/meshes/tools/welding_disk/disk.stl scale=0.001 0.001 0.001

File: backend/ros2_ws/eRob_moveit/src/eRob_ROS2_MoveIt/zeroerr/config/urdfs/erob_arm_family_motor_masses.urdf (robot description, URDF)
Before this commit: robot eRobo3, 12 links, 11 joints
Links:
- link Link_1: geometry collision mesh filename=package://zeroerr/meshes/robots/zeroerr/common/Link_1.stl scale=1.00000 1.00000 1.00000; visual mesh filename=package://zeroerr/meshes/robots/zeroerr/common/Link_1.stl scale=1.00000 1.00000 1.00000
- link Link_2: geometry collision mesh filename=package://zeroerr/meshes/robots/zeroerr/extended_links/Link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 scale=1.00000 1.00000 1.00000; visual mesh filename=package://zeroerr/meshes/robots/zeroerr/extended_links/Link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 scale=1.00000 1.00000 1.00000
- link Link_3: geometry collision mesh filename=package://zeroerr/meshes/robots/zeroerr/extended_links/Link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 scale=1.00000 1.00000 1.00000; visual mesh filename=package://zeroerr/meshes/robots/zeroerr/extended_links/Link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 scale=1.00000 1.00000 1.00000
- link Link_4: geometry collision mesh filename=package://zeroerr/meshes/robots/zeroerr/common/Link_4.stl scale=1.00000 1.00000 1.00000; visual mesh filename=package://zeroerr/meshes/robots/zeroerr/common/Link_4.stl scale=1.00000 1.00000 1.00000
- link Link_5: geometry collision mesh filename=package://zeroerr/meshes/robots/zeroerr/common/Link_5.stl scale=1.00000 1.00000 1.00000; visual mesh filename=package://zeroerr/meshes/robots/zeroerr/common/Link_5.stl scale=1.00000 1.00000 1.00000
- link Link_6: geometry collision mesh filename=package://zeroerr/meshes/robots/zeroerr/common/Link_6.stl scale=1.00000 1.00000 1.00000; visual mesh filename=package://zeroerr/meshes/robots/zeroerr/common/Link_6.stl scale=1.00000 1.00000 1.00000
- link base_link_inertial: geometry collision mesh filename=package://zeroerr/meshes/robots/zeroerr/common/base_link.stl scale=1.00000 1.00000 1.00000; visual mesh filename=package://zeroerr/meshes/robots/zeroerr/common/base_link.stl scale=1.00000 1.00000 1.00000
- link disk_link: geometry collision mesh filename=package://zeroerr/meshes/tools/welding_disk/disk.stl scale=0.001 0.001 0.001; visual mesh filename=package://zeroerr/meshes/tools/welding_disk/disk.stl scale=0.001 0.001 0.001

File: backend/ros2_ws/eRob_moveit/src/eRob_ROS2_MoveIt/zeroerr/config/urdfs/erob_arm_small.urdf (robot description, URDF)
Before this commit: robot eRobo3, 13 links, 12 joints
Links:
- link Link_1: geometry collision mesh filename=package://zeroerr/meshes/robots/zeroerr/common/Link_1.stl scale=1.00000 1.00000 1.00000; visual mesh filename=package://zeroerr/meshes/robots/zeroerr/common/Link_1.stl scale=1.00000 1.00000 1.00000
- link Link_2: geometry collision mesh filename=package://zeroerr/meshes/robots/zeroerr/short_links/Link_2.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 scale=1.00000 1.00000 1.00000; visual mesh filename=package://zeroerr/meshes/robots/zeroerr/short_links/Link_2.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 scale=1.00000 1.00000 1.00000
- link Link_3: geometry collision mesh filename=package://zeroerr/meshes/robots/zeroerr/short_links/Link_3.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 scale=1.00000 1.00000 1.00000; visual mesh filename=package://zeroerr/meshes/robots/zeroerr/short_links/Link_3.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 scale=1.00000 1.00000 1.00000
- link Link_4: geometry collision mesh filename=package://zeroerr/meshes/robots/zeroerr/common/Link_4.stl scale=1.00000 1.00000 1.00000; visual mesh filename=package://zeroerr/meshes/robots/zeroerr/common/Link_4.stl scale=1.00000 1.00000 1.00000
- link Link_5: geometry collision mesh filename=package://zeroerr/meshes/robots/zeroerr/common/Link_5.stl scale=1.00000 1.00000 1.00000; visual mesh filename=package://zeroerr/meshes/robots/zeroerr/common/Link_5.stl scale=1.00000 1.00000 1.00000
- link Link_6: geometry collision mesh filename=package://zeroerr/meshes/robots/zeroerr/common/Link_6.stl scale=1.00000 1.00000 1.00000; visual mesh filename=package://zeroerr/meshes/robots/zeroerr/common/Link_6.stl scale=1.00000 1.00000 1.00000
- link base_link_inertial: geometry collision mesh filename=package://zeroerr/meshes/robots/zeroerr/common/base_link.stl scale=1.00000 1.00000 1.00000; visual mesh filename=package://zeroerr/meshes/robots/zeroerr/common/base_link.stl scale=1.00000 1.00000 1.00000
- link tcp: geometry collision mesh filename=package://zeroerr/meshes/tools/pointer/ToolPointer.stl scale=0.001 0.001 0.001; visual sphere radius=0.00050
- link tool0: geometry collision mesh filename=package://zeroerr/meshes/tools/pointer/ToolPointer.stl scale=0.001 0.001 0.001; visual mesh filename=package://zeroerr/meshes/tools/pointer/ToolPointer.stl scale=0.001 0.001 0.001
