Commit message: Add backend cell-scene management and scene-editor controls; refine motion readiness and tolerances
git-svn-id: https://192.168.2.101:8443/svn/25488_ZeroErr/trunk@100 4fd3d927-d0b4-2643-a258-f5eadda0d283

File: backend/ros2_ws/eRob_moveit/src/eRob_ROS2_MoveIt/zeroerr/config/shared/cells/paint_tray_dry_compact.xacro (robot description, xacro)
@@ -14,12 +14,5 @@
         </material>
       </visual>
-      <!-- Include the simplified fixtures and equipment above the stepped
-           surfaces; the surface-only mesh omits these collision obstacles. -->
-      <collision>
-        <origin xyz="0 0 0" rpy="0 0 0" />
-        <geometry>
-          <mesh filename="package://zeroerr/meshes/cells/paint_tray_dry_compact/paint_tray_dry_compact.surface_3levels_above.stl" scale="0.001 0.001 0.001" />
-        </geometry>
-      </collision>
+      <!-- Cell collision geometry is profile-owned MoveIt world objects. -->
     </link>
     <joint name="mounting_surface_joint" type="fixed">
